File: keyboard.kicad_pcb (KiCad board)
At the start: 2 copper layers, 110 parts, among them SW1 SW_Push, SW10 SW_Push, SW11 SW_Push, SW12 SW_Push, SW13 SW_Push, SW14 SW_Push, SW15 SW_Push, SW16 SW_Push, SW17 SW_Push, SW18 SW_Push, SW19 SW_Push, SW2 SW_Push, SW20 SW_Push, SW21 SW_Push, SW22 SW_Push, SW23 SW_Push, SW24 SW_Push, SW25 SW_Push, SW26 SW_Push, SW27 SW_Push, SW28 SW_Push, SW29 SW_Push, SW3 SW_Push, SW30 SW_Push, SW31 SW_Push, SW32 SW_Push, SW33 SW_Push, SW34 SW_Push, SW35 SW_Push, SW36 SW_Push, SW37 SW_Push, SW38 SW_Push, SW39 SW_Push, SW4 SW_Push, SW40 SW_Push, SW41 SW_Push, SW42 SW_Push, SW43 SW_Push, SW44 SW_Push, SW45 SW_Push, SW46 SW_Push, SW47 SW_Push, SW48 SW_Push, SW49 SW_Push, SW5 SW_Push, SW50 SW_Push, SW51 SW_Push, SW52 SW_Push, SW6 SW_Push, SW7 SW_Push, SW8 SW_Push, SW9 SW_Push

Commit message: Added hardware source files and configure gitignore
Parts:
- removed H5: MountingHole, Panelization:mouse-bite-5mm-slot
- moved H3 290.2 mm to (36.9, 128.3), turned to 90 degrees
- moved SW11 195.2 mm to (241.3, 68.6)
- moved D11 192.2 mm to (240.0, 64.4), turned to 180 degrees
- moved SW49 184.3 mm to (222.2, 125.7)
- moved D49 178.5 mm to (221.0, 121.5), turned to 180 degrees
- moved SW24 171.3 mm to (241.3, 87.6)
- moved D42 170.2 mm to (87.6, 121.5), turned to 180 degrees
- moved D24 167.7 mm to (240.0, 83.4), turned to 180 degrees
- moved SW42 166.3 mm to (88.9, 125.7)
- moved D4 165.9 mm to (106.7, 64.4), turned to 180 degrees
- moved SW4 158.9 mm to (108.0, 68.6)
- moved SW37 148.5 mm to (241.3, 106.7)
- moved D29 147.7 mm to (87.6, 102.5), turned to 180 degrees
- moved D37 144.0 mm to (240.0, 102.5), turned to 180 degrees
- moved SW29 143.0 mm to (88.9, 106.7)
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- renumbered D37 to D10, D41 to D11, D45 to D12, D49 to D13, D2 to D14, D6 to D15, D10 to D16, D14 to D17, D22 to D19, D5 to D2, D26 to D20, D30 to D21, D34 to D22, D38 to D23, D42 to D24, D46 to D25, D50 to D26, D3 to D27, D7 to D28, D11 to D29, D9 to D3, D15 to D30, D19 to D31, D23 to D32, D27 to D33, D31 to D34, D39 to D36, D43 to D37, D47 to D38, D51 to D39, D13 to D4, D4 to D40, D8 to D41, D12 to D42, D16 to D43, D20 to D44, D24 to D45, D28 to D46, D32 to D47, D36 to D48, D40 to D49, D17 to D5, D44 to D50, D48 to D51, D21 to D6, D25 to D7, D29 to D8, D33 to D9, SW37 to SW10, SW41 to SW11, SW45 to SW12, SW49 to SW13, SW2 to SW14, SW6 to SW15, SW10 to SW16, SW14 to SW17, SW22 to SW19, SW5 to SW2, SW26 to SW20, SW30 to SW21, SW34 to SW22, SW38 to SW23, SW42 to SW24, SW46 to SW25, SW50 to SW26, SW3 to SW27, SW7 to SW28, SW11 to SW29, SW9 to SW3, SW15 to SW30, SW19 to SW31, SW23 to SW32, SW27 to SW33, SW31 to SW34, SW39 to SW36, SW43 to SW37, SW47 to SW38, SW51 to SW39, SW13 to SW4, SW4 to SW40, SW8 to SW41, SW12 to SW42, SW16 to SW43, SW20 to SW44, SW24 to SW45, SW28 to SW46, SW32 to SW47, SW36 to SW48, SW40 to SW49, SW17 to SW5, SW44 to SW50, SW48 to SW51, SW21 to SW6, SW25 to SW7, SW29 to SW8, SW33 to SW9
Connections:
- A1 pad 17: /COL11 -> /COL12
- A1 pad 18: /COL12 -> /COL11
Routing:
- net /ROW3: track 0.00 -> 337.6 mm, vias 0 -> 4
- net /ROW2: track 0.00 -> 335.3 mm, vias 0 -> 2
- net /ROW1: track 0.00 -> 289.8 mm, vias 0 -> 2
- net /ROW0: track 0.00 -> 268.7 mm
- net /COL1: track 47.4 -> 159.1 mm
- net /COL11: track 47.4 -> 155.6 mm
- net /COL3: track 31.6 -> 129.5 mm
- net /COL2: track 47.4 -> 142.6 mm
- net /COL12: track 89.0 -> 168.4 mm
- net /COL10: track 47.4 -> 119.6 mm
- net /COL4: track 47.4 -> 109.7 mm
- net /COL9: track 45.0 -> 104.6 mm
- net /COL0: track 233.4 -> 175.7 mm
- net /COL5: track 47.4 -> 93.1 mm
- net /COL8: track 47.4 -> 87.6 mm
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Other:
- board outline added: 264.8 x 106.7 mm

Commit message: Moved ESP to the left for charging
Parts:
- moved H4 267.4 mm to (305.5, 42.5)
- moved A1 114.9 mm to (38.7, 52.1)
Routing:
- net /COL10: track 119.6 -> 256.1 mm
- net /COL9: track 104.6 -> 239.1 mm
- net /COL8: track 87.6 -> 217.8 mm
- net /COL12: track 168.4 -> 297.5 mm
- net /COL11: track 155.6 -> 279.5 mm
- net /COL7: track 77.9 -> 199.5 mm
- net /COL6: track 81.0 -> 185.8 mm
- net /COL0: track 175.7 -> 79.2 mm
- net /COL5: track 93.1 -> 165.9 mm
- net /COL1: track 159.1 -> 93.9 mm
- net /ROW3: track 337.6 -> 385.9 mm, vias 4 -> 0
- net /COL4: track 109.7 -> 143.0 mm
- net /ROW1: track 289.8 -> 322.7 mm, vias 2 -> 0
- net /COL2: track 142.6 -> 110.4 mm
- net /ROW0: track 268.7 -> 298.2 mm
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Other:
- board size 264.8 x 106.7 mm -> 264.8 x 109.2 mm
