File: Hardware/keyboard.kicad_pcb (KiCad board)
At the start: 2 copper layers, 264.8 x 109.2 mm, 108 parts, among them SW1 SW_Push, SW10 SW_Push, SW11 SW_Push, SW12 SW_Push, SW13 SW_Push, SW14 SW_Push, SW15 SW_Push, SW16 SW_Push, SW17 SW_Push, SW18 SW_Push, SW19 SW_Push, SW2 SW_Push, SW20 SW_Push, SW21 SW_Push, SW22 SW_Push, SW23 SW_Push, SW24 SW_Push, SW25 SW_Push, SW26 SW_Push, SW27 SW_Push, SW28 SW_Push, SW29 SW_Push, SW3 SW_Push, SW30 SW_Push, SW31 SW_Push, SW32 SW_Push, SW33 SW_Push, SW34 SW_Push, SW35 SW_Push, SW36 SW_Push, SW37 SW_Push, SW38 SW_Push, SW39 SW_Push, SW4 SW_Push, SW40 SW_Push, SW41 SW_Push, SW42 SW_Push, SW43 SW_Push, SW44 SW_Push, SW45 SW_Push, SW46 SW_Push, SW47 SW_Push, SW48 SW_Push, SW49 SW_Push, SW5 SW_Push, SW50 SW_Push, SW51 SW_Push, SW52 SW_Push, SW6 SW_Push, SW7 SW_Push, SW8 SW_Push, SW9 SW_Push

Commit message: Fixed model by the requirements check
Parts:
- H1, H2, H3: footprint Panelization:mouse-bite-5mm-slot -> MountingHole:MountingHole_2.1mm
- SW1, SW10, SW11, SW12, SW13, SW14, SW15, SW16, SW17, SW18, SW19, SW2, SW20, SW21, SW22, SW23, SW24, SW25, SW26, SW27, SW28, SW29, SW3, SW30, SW31, SW32, SW33, SW34, SW35, SW36, SW37, SW38, SW39, SW4, SW40, SW41, SW42, SW43, SW44, SW45, SW46, SW47, SW48, SW49, SW5, SW50, SW51, SW52, SW6, SW7, SW8, SW9: moved to B.Cu
- moved D38 9.99 mm to (264.8, 110.7), turned to 90 degrees
- moved D39 9.99 mm to (283.8, 110.7), turned to 90 degrees
- moved D12 9.99 mm to (264.8, 72.6), turned to 90 degrees
- moved D13 9.99 mm to (283.8, 72.6), turned to 90 degrees
- moved D25 9.99 mm to (264.8, 91.6), turned to 90 degrees
- moved D26 9.99 mm to (283.8, 91.6), turned to 90 degrees
- moved D28 9.99 mm to (74.3, 110.7), turned to 90 degrees
- moved D29 9.99 mm to (93.3, 110.7), turned to 90 degrees
- moved D32 9.99 mm to (150.5, 110.7), turned to 90 degrees
- moved D34 9.99 mm to (188.6, 110.7), turned to 90 degrees
- moved D35 9.99 mm to (207.6, 110.7), turned to 90 degrees
- moved D36 9.99 mm to (226.7, 110.7), turned to 90 degrees
- moved D37 9.99 mm to (245.7, 110.7), turned to 90 degrees
- moved D27 9.99 mm to (55.2, 110.7), turned to 90 degrees
- moved D51 9.99 mm to (264.8, 129.7), turned to 90 degrees
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Routing:
- net /COL10: track 256.1 -> 230.6 mm, vias 0 -> 6
- net /COL9: track 239.1 -> 214.1 mm, vias 0 -> 6
- net /COL6: track 185.8 -> 164.6 mm, vias 0 -> 6
- net /COL12: track 297.5 -> 277.1 mm
- net /COL8: track 217.8 -> 197.6 mm, vias 0 -> 6
- net /COL11: track 279.5 -> 260.6 mm, vias 0 -> 6
- net /COL7: track 199.5 -> 181.1 mm, vias 0 -> 6
- net /COL5: track 165.9 -> 148.1 mm, vias 0 -> 6
- net Net-(D27-A): track 11.3 -> 27.3 mm, vias 0 -> 2
- net Net-(D14-A): track 11.3 -> 27.3 mm, vias 0 -> 2
- net Net-(D1-A): track 11.3 -> 26.5 mm, vias 0 -> 2
- net /COL3: track 129.9 -> 117.8 mm, vias 0 -> 6
- net /COL4: track 143.0 -> 131.6 mm, vias 0 -> 6
- net /COL1: track 93.9 -> 84.0 mm, vias 0 -> 6
- net /COL2: track 110.4 -> 101.2 mm, vias 0 -> 6
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