File: Hardware/keyboard.kicad_sch (KiCad schematic)
At the start: 115 parts, among them SW1 SW_Push, SW10 SW_Push, SW11 SW_Push, SW12 SW_Push, SW13 SW_Push, SW14 SW_Push, SW15 SW_Push, SW16 SW_Push, SW17 SW_Push, SW18 SW_Push, SW19 SW_Push, SW2 SW_Push, SW20 SW_Push, SW21 SW_Push, SW22 SW_Push, SW23 SW_Push, SW24 SW_Push, SW25 SW_Push, SW26 SW_Push, SW27 SW_Push, SW28 SW_Push, SW29 SW_Push, SW3 SW_Push, SW30 SW_Push, SW31 SW_Push, SW32 SW_Push, SW33 SW_Push, SW34 SW_Push, SW35 SW_Push, SW36 SW_Push, SW37 SW_Push, SW38 SW_Push, SW39 SW_Push, SW4 SW_Push, SW40 SW_Push, SW41 SW_Push, SW42 SW_Push, SW43 SW_Push, SW44 SW_Push, SW45 SW_Push, SW46 SW_Push, SW47 SW_Push, SW48 SW_Push, SW49 SW_Push, SW5 SW_Push, SW50 SW_Push, SW51 SW_Push, SW52 SW_Push, SW6 SW_Push, SW7 SW_Push, SW8 SW_Push, SW9 SW_Push, U1 XIAO-nRF52840-SMD, U2 ESP32-WROOM-E

Commit message: Finihed Case Design
Parts:
- removed H5: MountingHole, Panelization:mouse-bite-5mm-slot, symbol Mechanical:MountingHole
- removed R1: 806k, Resistor_SMD:R_0805_2012Metric, symbol Device:R
- removed R2: 2M, Resistor_SMD:R_0805_2012Metric, symbol Device:R
- removed TP1: BAT, TestPoint:TestPoint_Pad_D2.0mm, symbol Connector:TestPoint
- removed TP2: GND, TestPoint:TestPoint_Pad_D2.0mm, symbol Connector:TestPoint
- removed U1: XIAO-nRF52840-SMD, XIAO:modified-XIAO-nRF52840-SMD, symbol Seeed_Studio_XIAO_Series:XIAO-nRF52840-SMD
- removed U2: ESP32-WROOM-E, PCM_Espressif:ESP32-WROOM-32E, symbol Espressif:ESP32-WROOM-E
- added A1: Adafruit_Feather_HUZZAH32_ESP32, Module:Adafruit_Feather, symbol Custom_ESP32_Library:Adafruit_Feather_HUZZAH32_ESP32
- renumbered D37 to D10, D41 to D11, D45 to D12, D49 to D13, D2 to D14, D6 to D15, D10 to D16, D14 to D17, D22 to D19, D5 to D2, D26 to D20, D30 to D21, D34 to D22, D38 to D23, D42 to D24, D46 to D25, D50 to D26, D3 to D27, D7 to D28, D11 to D29, D9 to D3, D15 to D30, D19 to D31, D23 to D32, D27 to D33, D31 to D34, D39 to D36, D43 to D37, D47 to D38, D51 to D39, D13 to D4, D4 to D40, D8 to D41, D12 to D42, D16 to D43, D20 to D44, D24 to D45, D28 to D46, D32 to D47, D36 to D48, D40 to D49, D17 to D5, D44 to D50, D48 to D51, D21 to D6, D25 to D7, D29 to D8, D33 to D9, SW37 to SW10, SW41 to SW11, SW45 to SW12, SW49 to SW13, SW2 to SW14, SW6 to SW15, SW10 to SW16, SW14 to SW17, SW22 to SW19, SW5 to SW2, SW26 to SW20, SW30 to SW21, SW34 to SW22, SW38 to SW23, SW42 to SW24, SW46 to SW25, SW50 to SW26, SW3 to SW27, SW7 to SW28, SW11 to SW29, SW9 to SW3, SW15 to SW30, SW19 to SW31, SW23 to SW32, SW27 to SW33, SW31 to SW34, SW39 to SW36, SW43 to SW37, SW47 to SW38, SW51 to SW39, SW13 to SW4, SW4 to SW40, SW8 to SW41, SW12 to SW42, SW16 to SW43, SW20 to SW44, SW24 to SW45, SW28 to SW46, SW32 to SW47, SW36 to SW48, SW40 to SW49, SW17 to SW5, SW44 to SW50, SW48 to SW51, SW21 to SW6, SW25 to SW7, SW29 to SW8, SW33 to SW9
Connections:
- net COL0: now also A1.6 (A0/IO26)
- net COL1: now also A1.7 (A1/IO25)
- net COL10: now also A1.16 (TX/IO17)
- net COL11: now also A1.18 (SCL/IO22)
- net COL12: now also A1.17 (SDA/IO23)
- net COL2: now also A1.8 (A2/IO34(IN))
- net COL3: now also A1.9 (A3/IO39(IN))
- net COL4: now also A1.10 (A4/IO36(IN))
- net COL5: now also A1.11 (A5/IO4)
- net COL6: now also A1.12 (SCK/IO5)
- net COL7: now also A1.13 (MOSI/IO18)
- net COL8: now also A1.14 (MISO/IO19)
- net COL9: now also A1.15 (RX/IO16)
- net GND: now also A1.27 (GND)
- net ROW0: now also A1.26 (D21/IO21)
- net ROW1: now also A1.25 (D14/IO14)
- net ROW2: now also A1.24 (D32/IO32)
- net ROW3: now also A1.19 (D13/IO13)
- no-connect marks 8 -> 9
Other:
- note added: "ESP32 Feather Adafruit HUZZAH32"
- note removed: "Battery Sense"
- note removed: "Test Points"
- note removed: "xiao"
- moved on the sheet: D1, D10, D11, D12, D13, D14, D15, D16, D17, D18, D19, D2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

Commit message: Fixed model by the requirements check
Parts:
- removed H4: MountingHole, Panelization:mouse-bite-5mm-slot, symbol Mechanical:MountingHole
- H1, H2, H3: footprint Panelization:mouse-bite-5mm-slot -> MountingHole:MountingHole_2.1mm
Changed lines of the file:
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@@
 			)
 		)
-		(property "Footprint" "Panelization:mouse-bite-5mm-slot"
+		(property "Footprint" "MountingHole:MountingHole_2.1mm"
 			(at 132.08 181.61 0)
 			(effects
@@
 	)
 	(symbol
-		(lib_id "Mechanical:MountingHole")
-		(at 158.75 181.61 0)
-		(unit 1)
-		(exclude_from_sim no)
-		(in_bom no)
-		(on_board yes)
-		(dnp no)
-		(property "Reference" "H4"
-			(at 161.29 181.6099 0)
-			(effects
-				(font
-					(size 1.27 1.27)
-				)
-				(justify left)
-			)
-		)
-		(property "Value" "MountingHole"
-			(at 161.29 182.8799 0)
-			(effects
-				(font
-					(size 1.27 1.27)
-				)
-				(justify left)
-				(hide yes)
-			)
-		)
-		(property "Footprint" "Panelization:mouse-bite-5mm-slot"
-			(at 158.75 181.61 0)
-			(effects
-				(font
-					(size 1.27 1.27)
-				)
-				(hide yes)
-			)
-		)
-		(property "Datasheet" "~"
-			(at 158.75 181.61 0)
-			(effects
-				(font
-					(size 1.27 1.27)
-				)
-				(hide yes)
-			)
-		)
-		(property "Description" "Mounting Hole without connection"
-			(at 158.75 181.61 0)
-			(effects
-				(font
-					(size 1.27 1.27)
-				)
-				(hide yes)
-			)
-		)
-		(instances
-			(project "keyboard"
-				(path "/76daee2a-e779-4aa0-aa95-eaf0bba9e97a"
-					(reference "H4")
-					(unit 1)
-				)
-			)
-		)
-	)
-	(symbol
 		(lib_id "Switch:SW_Push")
 		(at 237.49 87.63 0)
@@
 			)
 		)
-		(property "Footprint" "Panelization:mouse-bite-5mm-slot"
+		(property "Footprint" "MountingHole:MountingHole_2.1mm"
 			(at 140.97 181.61 0)
 			(effects
@@
 			)
 		)
-		(property "Footprint" "Panelization:mouse-bite-5mm-slot"
+		(property "Footprint" "MountingHole:MountingHole_2.1mm"
 			(at 149.86 181.61 0)
 			(effects
